File: ClockGenIC.kicad_sch (KiCad schematic)
At the start: 8 parts, among them J5 Conn_Coaxial, U1 ADF4351

Commit message: Fix: replaced deleted stuff
lost some components in the last merge so this is replacing them
Parts:
- added U5: ADF4351BCPZ-RL7, CP_32_7_ADI, symbol ADF4351BCPZ-RL7:ADF4351BCPZ-RL7
Changed lines of the file:
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@@
+	)
+	(symbol
+		(lib_id "ADF4351BCPZ-RL7:ADF4351BCPZ-RL7")
+		(at 182.88 59.69 0)
+		(unit 1)
+		(exclude_from_sim no)
+		(in_bom yes)
+		(on_board yes)
+		(dnp no)
+		(fields_autoplaced yes)
+		(property "Reference" "U5"
+			(at 208.28 49.53 0)
+			(effects
+				(font
+					(size 1.524 1.524)
+				)
+			)
+		)
+		(property "Value" "ADF4351BCPZ-RL7"
+			(at 208.28 52.07 0)
+			(effects
+				(font
+					(size 1.524 1.524)
+				)
+			)
+		)
+		(property "Footprint" "CP_32_7_ADI"
+			(at 182.88 59.69 0)
+			(effects
+				(font
+					(size 1.27 1.27)
+					(italic yes)
+				)
+				(hide yes)
+			)
+		)
+		(property "Datasheet" "https://www.analog.com/media/en/technical-documentation/data-sheets/ADF4351.pdf"
+			(at 182.88 59.69 0)
+			(effects
+				(font
+					(size 1.27 1.27)
+					(italic yes)
+				)
+				(hide yes)
+			)
+		)
+		(property "Description" ""
+			(at 182.88 59.69 0)
+			(effects
+				(font
+					(size 1.27 1.27)
+				)
+				(hide yes)
+			)
+		)
+		(pin "7"
+		)
+		(pin "9"
+		)
+		(pin "31"
+		)
+		(pin "28"
+		)
+		(pin "15"
+		)
+		(pin "25"
+		)
+		(pin "29"
+		)
+		(pin "3"
+		)
+		(pin "13"
+		)
+		(pin "14"
+		)
+		(pin "33"
+		)
+		(pin "32"
+		)
+		(pin "11"
+		)
+		(pin "2"
+		)
+		(pin "12"
+		)
+		(pin "1"
+		)
+		(pin "4"
+		)
+		(pin "5"
+		)
+		(pin "16"
+		)
+		(pin "6"
+		)
+		(pin "8"
+		)
+		(pin "10"
+		)
+		(pin "30"
+		)
+		(pin "27"
+		)
+		(pin "26"
+		)
+		(pin "22"
+		)
+		(pin "21"
+		)
+		(pin "18"
+		)
+		(pin "19"
+		)
+		(pin "17"
+		)
+		(pin "20"
+		)
+		(pin "24"
+		)
+		(pin "23"
+		)
+		(instances
+			(project ""
+				(path "/e1444a2d-a0c4-493c-a136-c624dc084e46/5eadf96c-4633-4d78-8a47-09b3347a9db0"
+					(reference "U5")
+					(unit 1)
+				)
+			)
+		)
 	)
 	(symbol

Commit message: IC update
Parts:
- removed U5: ADF4351BCPZ-RL7, CP_32_7_ADI, symbol ADF4351BCPZ-RL7:ADF4351BCPZ-RL7
- added C13: 10pF, Capacitor_SMD:C_0603_1608Metric_Pad1.08x0.95mm_HandSolder, symbol Device:C
- added C14, C2: 1n, Capacitor_SMD:C_0603_1608Metric_Pad1.08x0.95mm_HandSolder, symbol Device:C
- added C15, C16: 0.1uF, Capacitor_SMD:C_0603_1608Metric_Pad1.08x0.95mm_HandSolder, symbol Device:C
- added J4, J6: Conn_Coaxial, Connector_Coaxial:SMA_Samtec_SMA-J-P-H-ST-EM1_EdgeMount, symbol Connector:Conn_Coaxial
- added L1, L2: 3.9n, symbol Device:L
- added R1: 1k, symbol Device:R
- added R11: 4.7k, symbol Device:R
- added R12, R3: 51, Resistor_SMD:R_0603_1608Metric_Pad0.98x0.95mm_HandSolder, symbol Device:R
- added R2: 51, symbol Device:R
- added U2: AP2112K-3.3, Package_TO_SOT_SMD:SOT-23-5, symbol Regulator_Linear:AP2112K-3.3
- added Y2: TG2520SMN-xx.xxxxxxMhz-xxxxNM, Oscillator:Oscillator_SMD_SeikoEpson_TG2520SMN-xxx-xxxxxx-4Pin_2.5x2.0mm, symbol Oscillator:TG2520SMN-xx.xxxxxxMhz-xxxxNM
- R7: value 750 -> 390
Connections:
- net 3.3V: now also U1.28 (DVDD), U1.32 (SDVDD), R1.1
- net CPout: now also C9.1; no longer R7.2
- net GND: now also R7.1, U1.11 (AGNDVCO), U1.18 (AGNDVCO), U1.21 (AGNDVCO), U1.27 (DGND), U1.31 (SDGND), U1.33 (EP), U1.8 (CPGND), J4.2 (Ext), R11.2, R12.2, R2.2, R3.2, U2.2 (GND), Y2.2 (GND); no longer C9.2
- net REFIN: now also C16.1
- net RF_OUT_A+: now also C14.2, L2.2
- net RF_OUT_A-: now also C13.2, C2.2, L1.2
- net VTUNE: now also U1.20 (VTUNE)
- net VVCO: now reaches U1.16 (VVCO)
- net VVCO: now also U1.17 (VVCO), L1.1, L2.1, U2.5 (VOUT)
- net at U1.22 (RSET): now also R11.1
- net LD: now reaches U1.25 (LD)
- new net: C9.2, R7.2
- new net: C15.1, C16.2, R2.1
- new net: J6.1 (In), Y2.3 (OUT)
- new net: R1.2, Y2.4 (Vcc)
- new net: C13.1, J4.1 (In)
- new net: C14.1, R12.1
- new net: C2.1, R3.1
- new net: C15.2, J6.2 (Ext)
- new net +5V: U2.1 (VIN), U2.3 (EN)
Other:
- moved on the sheet: C10, C7, C8, C9, J5, R7, R8
